File: Design/Hardware/Design Files/AL.kicad_pcb (KiCad board)
At the start: 2 copper layers, 22 parts, among them J1 Screw_Terminal_01x02, J2 Conn_01x04, J3 Screw_Terminal_01x02, M1 IFX9201SG, U1 AP2204RB-3.3, U2 STM8L051F3

Commit message: Schematic Update
Parts:
- removed D1: SMBJ12CA, AL:DO214AA
- removed J3: Screw_Terminal_01x02, Connectors_Terminal_Blocks:TerminalBlock_bornier-2_P5.08mm
- added C10: 100n, Capacitors_SMD:C_0603_HandSoldering, F.Cu at (109.7, 79.7)
- added C11: 100n, Capacitors_SMD:C_0603_HandSoldering, F.Cu at (131.0, 68.4)
- added C12: 1u, Capacitors_SMD:C_0603_HandSoldering, F.Cu at (117.9, 79.2)
- added C13: 4.7u, Capacitors_SMD:C_0603_HandSoldering, F.Cu at (122.7, 74.4)
- added C14: 2.2u, Capacitors_SMD:C_0603_HandSoldering, F.Cu at (126.9, 68.4)
- added C15: 1u, Capacitors_SMD:C_0603_HandSoldering, F.Cu at (130.9, 63.6)
- added C16: 1u, Capacitors_SMD:C_0603_HandSoldering, F.Cu at (126.9, 63.6)
- added C17: 100n, Capacitors_SMD:C_0603_HandSoldering, F.Cu at (105.6, 78.3)
- added C18: 0.1u, Capacitors_SMD:C_0603_HandSoldering, F.Cu at (122.7, 69.6)
- added C19: 2.2u, Capacitors_SMD:C_0603_HandSoldering, F.Cu at (113.8, 79.7)
- added C20: 10n, Capacitors_SMD:C_0603_HandSoldering, F.Cu at (130.9, 58.8)
- added C21: 10n, Capacitors_SMD:C_0603_HandSoldering, F.Cu at (105.5, 73.5)
- added D4: SMBJ12CA, AL:DO214AA, F.Cu at (59.9, 83.4)
- added D5: TS4148C, Diodes_SMD:D_0603, F.Cu at (99.2, 68.1)
- added D6: BAT54C, TO_SOT_Packages_SMD:TSOT-23, F.Cu at (118.5, 44.1)
- added F1: F1 LF-2920L, Fuse_Holders_and_Fuses:Fuse_SMD2920, F.Cu at (101.7, 60.3)
- added J4: Screw_Terminal_01x02, TerminalBlocks_Phoenix:TerminalBlock_Phoenix_MKDS1.5-2pol, F.Cu at (62.0, 62.8)
- added Q1: NX7002, TO_SOT_Packages_SMD:TSOT-23, F.Cu at (75.4, 81.6)
- added Q2: FDD6637, TO_SOT_Packages_SMD:TO-252-2, F.Cu at (109.8, 46.1)
- added Q3: FDD6637, TO_SOT_Packages_SMD:TO-252-2, F.Cu at (78.9, 72.6)
- added Q4: NX7002, TO_SOT_Packages_SMD:TSOT-23, F.Cu at (81.6, 81.6)
- added R10: 100, Resistors_SMD:R_0603_HandSoldering, F.Cu at (101.3, 73.7)
- added R11: 10k, Resistors_SMD:R_0603_HandSoldering, F.Cu at (129.6, 54.0)
- added R12: 0, Resistors_SMD:R_0805_HandSoldering, F.Cu at (128.8, 43.3)
- added R14: 1M, Resistors_SMD:R_0603_HandSoldering, F.Cu at (123.6, 48.9)
- added R15: 100, Resistors_SMD:R_0603_HandSoldering, F.Cu at (128.0, 48.9)
- added R16: 470k, Resistors_SMD:R_0603_HandSoldering, F.Cu at (113.9, 60.0)
- added R17: 1M, Resistors_SMD:R_0603_HandSoldering, F.Cu at (133.5, 43.1)
- added R18: 100, Resistors_SMD:R_0603_HandSoldering, F.Cu at (109.9, 65.0)
- added R19: 52.3k, Resistors_SMD:R_0603_HandSoldering, F.Cu at (114.4, 65.0)
- added R20: 82k, Resistors_SMD:R_0603_HandSoldering, F.Cu at (109.9, 70.1)
- added R21: 10, Resistors_SMD:R_0603_HandSoldering, F.Cu at (101.3, 78.7)
- added R22: 10k, Resistors_SMD:R_0603_HandSoldering, F.Cu at (125.2, 54.0)
- added R23: 10k, Resistors_SMD:R_0603_HandSoldering, F.Cu at (133.5, 48.1)
- added R24: 10k, Resistors_SMD:R_0603_HandSoldering, F.Cu at (122.6, 59.0)
- added R25: 10k, Resistors_SMD:R_0603_HandSoldering, F.Cu at (114.3, 70.1)
- added R26: 10k, Resistors_SMD:R_0603_HandSoldering, F.Cu at (118.3, 60.0)
- added R6: 100, Resistors_SMD:R_1206, F.Cu at (123.8, 43.5)
- added R7: 100, Resistors_SMD:R_1206, F.Cu at (116.3, 54.5)
- added R8: 100, Resistors_SMD:R_1206, F.Cu at (109.4, 59.4)
- added R9: 100, Resistors_SMD:R_1206, F.Cu at (96.7, 73.4)
- added U3: STM8L051F3, Housings_SSOP:SSOP-20_4.4x6.5mm_Pitch0.65mm, F.Cu at (89.5, 75.7)
- C1, C2: value 150uF/12V -> 100n; footprint Capacitors_THT:CP_Radial_D10.0mm_P5.00mm -> Capacitors_SMD:C_0603_HandSoldering
- C3, C8: value 1uF -> 100n; footprint Capacitors_SMD:C_0603 -> Capacitors_SMD:C_0603_HandSoldering
- C4, C7: value 10nF -> 1u; footprint Capacitors_SMD:C_0603 -> Capacitors_SMD:C_0603_HandSoldering
- C5: value 2.2uF -> 1u; footprint Capacitors_SMD:C_0603 -> Capacitors_SMD:C_0603_HandSoldering
- C6: value 0.1uF -> 1u; footprint Capacitors_SMD:C_0603 -> Capacitors_SMD:C_0603_HandSoldering
- C9: value 0.1uF -> 470p; footprint Capacitors_SMD:C_0603 -> Capacitors_SMD:C_0603_HandSoldering
- D2: value D_Schottky -> TS4148C; footprint Diodes_SMD:D_MiniMELF -> Diodes_SMD:D_0603
- J1: value Screw_Terminal_01x02 -> Screw_Terminal_01x06; footprint Connectors_Terminal_Blocks:TerminalBlock_bornier-2_P5.08mm -> TerminalBlocks_Phoenix:TerminalBlock_Phoenix_MKDS1.5-6pol
- J2: value Conn_01x04 -> Screw_Terminal_01x02; footprint Pin_Headers:Pin_Header_Straight_1x04_Pitch1.00mm -> TerminalBlocks_Phoenix:TerminalBlock_Phoenix_MKDS1.5-2pol
- R2: value 10k -> 0; footprint Resistors_SMD:R_0603 -> Resistors_SMD:R_0805_HandSoldering
- R3: value 10k -> 100; footprint Resistors_SMD:R_0603 -> Resistors_SMD:R_0603_HandSoldering
- R4: value 10k -> 1M; footprint Resistors_SMD:R_0603 -> Resistors_SMD:R_0603_HandSoldering
- R5: value 0 -> 0.005; footprint Resistors_SMD:R_0603 -> Resistors_SMD:R_2512_HandSoldering
- RV1: value 0-10k -> POT_TRIM; footprint Potentiometers:Potentiometer_Trimmer_Bourns_3339H_Horizontal -> Potentiometers:Potentiometer_Trimmer_Bourns_3339P_Horizontal
- U1: value AP2204RB-3.3 -> BQ76920; footprint TO_SOT_Packages_SMD:SOT-23-5 -> Housings_SSOP:SSOP-20_4.4x6.5mm_Pitch0.65mm
- U2: value STM8L051F3 -> AP2204K-ADJ; footprint Housings_SSOP:TSSOP-20_4.4x6.5mm_Pitch0.65mm -> TO_SOT_Packages_SMD:SOT-23-5
- moved C6 66.7 mm to (122.8, 63.9), turned to 0 degrees
- moved C2 63.1 mm to (118.7, 64.8), turned to 0 degrees
- moved C9 56.4 mm to (133.8, 53.0), turned to 0 degrees
- moved C5 56.2 mm to (113.8, 74.9)
- moved C7 54.5 mm to (118.7, 69.6)
- moved D2 51.4 mm to (110.4, 54.1), turned to 0 degrees
- moved C8 50.8 mm to (105.6, 83.1), turned to 0 degrees
- moved R4 48.8 mm to (120.8, 54.0), turned to 0 degrees
- moved C1 44.9 mm to (118.6, 74.4), turned to 0 degrees
- moved C4 40.0 mm to (126.8, 58.8)
- moved C3 37.7 mm to (109.7, 74.9), turned to 0 degrees
- moved R2 35.3 mm to (105.2, 68.4), turned to 0 degrees
- moved R3 34.8 mm to (96.5, 78.9)
- moved R5 34.7 mm to (90.6, 58.8), turned to 0 degrees
- moved U1 26.6 mm to (68.4, 75.0)
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Connections:
- C1 pad 1: OUT1 -> GND
- C1 pad 2: OUT2 -> BAT1N
- C2 pad 1: 12VDC -> GND
- C2 pad 2: PGND -> BATNOUT
- C3 pad 1: 12VDC -> BAT+
- C3 pad 2: GND -> Net-(C3-Pad2)
- C4 pad 1: OUT1 -> GND
- C4 pad 2: GND -> Net-(C4-Pad2)
- C5 pad 1: +3V3 -> Net-(C5-Pad1)
- C6 pad 1: 12VDC -> Net-(C6-Pad1)
- C6 pad 2: GND -> Net-(C6-Pad2)
- C7 pad 1: OUT2 -> Net-(C6-Pad2)
- C7 pad 2: GND -> Net-(C5-Pad1)
- C8 pad 1: GND -> Net-(C3-Pad2)
- C8 pad 2: 3V3 -> BATPOUT
- C9 pad 2: 3V3 -> Net-(C9-Pad2)
- D2 pad 1: 3V3 -> Net-(D2-Pad1)
- D2 pad 2: +3V3 -> BAT+
- J1 pad 1: 12VDC -> BAT1N
- J1 pad 2: PGND -> BAT1P
- J2 pad 1: 3V3 -> BATPOUT
- J2 pad 2: SWIM -> BATNOUT
- M1 pad 2: 3V3 -> VDD
- M1 pad 4: 12VDC -> BATPOUT
- R2 pad 1: 3V3 -> GND
- R2 pad 2: DIS -> BAT1N
- R3 pad 1: PWM -> Net-(Q1-Pad1)
- R3 pad 2: GND -> DSG
- R4 pad 1: 3V3 -> BAT+
- R4 pad 2: NSS -> Net-(Q1-Pad3)
- R5 pad 1: GND -> BATNOUT
- R5 pad 2: PGND -> BAT1N
- RV1 pad 1: 3V3 -> VDD
- U1 pad 1: +3V3 -> DSG
- U1 pad 2: GND -> CHG
- U1 pad 3: 12VDC -> Net-(C14-Pad2)
- U1 pad 4: (no net) -> SDA
- U1 pad 5: (no net) -> SCL
- U2 pad 1: Net-(U2-Pad1) -> BATPOUT
- U2 pad 2: Net-(U2-Pad2) -> GND
- U2 pad 3: SWIM -> BATPOUT
- U2 pad 4: RST -> Net-(R19-Pad2)
Routing:
- net +3V3: track 5.32 -> 0.00 mm
- net 3V3: track 3.01 -> 0.00 mm
Other:
- rule pad_to_mask_clearance: 0.2 -> 0
