File: Design/Hardware/Design Files/AL.sch (KiCad schematic (older format))
At the start: 23 parts, among them J1 Screw_Terminal_01x02, J2 Conn_01x04, J3 Screw_Terminal_01x02, M1 IFX9201SG, U1 AP2204RB-3.3, U2 STM8L051F3

Commit message: Schematic Update
Parts:
- removed C1, C2: 150uF/12V, Capacitors_THT:CP_Radial_D10.0mm_P5.00mm, symbol CP
- removed D1: SMBJ12CA, AL:DO214AA, symbol D_TVS
- removed D2: D_Schottky, Diodes_SMD:D_MiniMELF, symbol D_Schottky
- removed J1, J3: Screw_Terminal_01x02, Connectors_Terminal_Blocks:TerminalBlock_bornier-2_P5.08mm, symbol Screw_Terminal_01x02
- removed J2: Conn_01x04, Pin_Headers:Pin_Header_Straight_1x04_Pitch1.00mm, symbol Conn_01x04
- removed U1: AP2204RB-3.3, TO_SOT_Packages_SMD:SOT-89-3, symbol AP2204RB-3.3
- removed U2: STM8L051F3, Housings_SSOP:TSSOP-20_4.4x6.5mm_Pitch0.65mm, symbol STM8L051F3
- added C1, C10, C11, C17, C2: 100n, Capacitors_SMD:C_0603_HandSoldering, symbol C
- added C12, C15, C16: 1u, Capacitors_SMD:C_0603_HandSoldering, symbol C
- added C13: 4.7u, Capacitors_SMD:C_0603_HandSoldering, symbol C
- added C14, C19: 2.2u, Capacitors_SMD:C_0603_HandSoldering, symbol C
- added C18: 0.1u, Capacitors_SMD:C_0603_HandSoldering, symbol C
- added C20, C21: 10n, Capacitors_SMD:C_0603_HandSoldering, symbol C
- added D1, D3: 5.6V, symbol D_Schottky
- added D2, D5: TS4148C, Diodes_SMD:D_0603, symbol D
- added D4: SMBJ12CA, AL:DO214AA, symbol D_TVS
- added D6: BAT54C, TO_SOT_Packages_SMD:TSOT-23, symbol D_Schottky_x2_KCom_AAK
- added F1: F1 LF-2920L, Fuse_Holders_and_Fuses:Fuse_SMD2920, symbol Polyfuse_Small
- added J1: Screw_Terminal_01x06, symbol Screw_Terminal_01x06
- added J2, J4: Screw_Terminal_01x02, symbol Screw_Terminal_01x02
- added J3: Conn_01x04, symbol Conn_01x04
- added Q1, Q4: NX7002, TO_SOT_Packages_SMD:TSOT-23, symbol Q_NMOS_GSD
- added Q2, Q3: FDD6637, TO_SOT_Packages_SMD:TO-252-2, symbol Q_PMOS_GDS
- added R10, R15, R18: 100, Resistors_SMD:R_0603_HandSoldering, symbol R
- added R11, R22, R23, R24, R25, R26: 10k, Resistors_SMD:R_0603_HandSoldering, symbol R
- added R12: 0, Resistors_SMD:R_0805_HandSoldering, symbol R
- added R13: 100, symbol R
- added R14, R17: 1M, Resistors_SMD:R_0603_HandSoldering, symbol R
- added R16: 470k, Resistors_SMD:R_0603_HandSoldering, symbol R
- added R19: 52.3k, Resistors_SMD:R_0603_HandSoldering, symbol R
- added R20: 82k, Resistors_SMD:R_0603_HandSoldering, symbol R
- added R21: 10, Resistors_SMD:R_0603_HandSoldering, symbol R
- added R6, R7, R8, R9: 100, Resistors_SMD:R_1206, symbol R
- added U1: BQ76920, Housings_SSOP:SSOP-20_4.4x6.5mm_Pitch0.65mm, symbol BQ76920
- added U2: AP2204K-ADJ, TO_SOT_Packages_SMD:SOT-23-5, symbol AP2204K-ADJ
- added U3: STM8L051F3, Housings_SSOP:SSOP-20_4.4x6.5mm_Pitch0.65mm, symbol STM8L051F3
- C3, C8: value 1uF -> 100n; footprint Capacitors_SMD:C_0603 -> Capacitors_SMD:C_0603_HandSoldering
- C4, C7: value 10nF -> 1u; footprint Capacitors_SMD:C_0603 -> Capacitors_SMD:C_0603_HandSoldering
- C5: value 2.2uF -> 1u; footprint Capacitors_SMD:C_0603 -> Capacitors_SMD:C_0603_HandSoldering
- C6: value 0.1uF -> 1u; footprint Capacitors_SMD:C_0603 -> Capacitors_SMD:C_0603_HandSoldering
- C9: value 0.1uF -> 470p; footprint Capacitors_SMD:C_0603 -> Capacitors_SMD:C_0603_HandSoldering
- R1: value 10 -> 1M
- R2: value 10k -> 0; footprint Resistors_SMD:R_0603 -> Resistors_SMD:R_0805_HandSoldering
- R3: value 10k -> 100; footprint Resistors_SMD:R_0603 -> Resistors_SMD:R_0603_HandSoldering
- R4: value 10k -> 1M; footprint Resistors_SMD:R_0603 -> Resistors_SMD:R_0603_HandSoldering
- R5: value 0 -> 0.005; footprint Resistors_SMD:R_0603 -> Resistors_SMD:R_2512_HandSoldering; Power (none) -> 1.5W
- RV1: value 0-10k -> POT_TRIM; footprint Potentiometers:Potentiometer_Trimmer_Bourns_3339H_Horizontal -> Potentiometers:Potentiometer_Trimmer_Bourns_3339P_Horizontal
Connections:
- net ADC_IN: now also U3.13 (PB3)
- net CLK: now also U3.15 (PB5)
- net DIR: now also U3.11 (PB1)
- net DIS: now also R24.1, U3.12 (PB2); no longer R2.2
- net GND: now also C4.1, R2.1, C1.1, C15.2, C16.2, C17.2, C18.1, C19.2, C2.1, C20.1, C21.1, J3.3 (Pin_3), R12.1, R16.2, R20.2, R25.1, U2.2 (GND), U3.7 (VSS); no longer C3.2, C4.2, C6.2, C7.2, C8.1, R3.2, R5.1
- net NSS: now also R26.1, U3.14 (PB4); no longer R4.2
- net OUT1: now also C20.2, J4.1 (Pin_1); no longer C4.1
- net OUT2: now also C21.2, J4.2 (Pin_2); no longer C7.1
- net PWM: now also R25.2, U3.10 (PB0); no longer R3.1
- net RST: now also J3.4 (Pin_4), U3.4 (PA1/NRST)
- net SI: now also U3.16 (PB6)
- net SO: now also R21.2, U3.17 (PB7); no longer R1.2
- net SWIM: now also J3.2 (Pin_2), U3.3 (PA0)
- net at M1.3 (SO): now also R21.1; no longer R1.1
- net +3V3: no longer names the net of C5.1
- net +3V3: now also C7.2, R8.2, U1.16 (VC1)
- removed net 12VDC: C3.1, C6.1, M1.4 (VS)
- removed net 3V3: C8.2, C9.2, M1.2 (VSO), R2.1, R4.1, RV1.1
- net PGND renamed BAT1N
- net BAT1N: now also R2.2, C1.2, J1.1 (Pin_1), R9.1, U1.18 (SRP)
- new net: C9.2, R16.1, U1.20 (ALERT), U3.1 (PC5)
- new net: D5.2 (A), U3.20 (PC4)
- new net: C6.1, R6.2, U1.12 (VC5)
- new net: C6.2, C7.1, R7.2, U1.13 (VC4), U1.14 (VC3), U1.15 (VC2)
- new net: C12.1, U1.7 (CAP1)
- new net: Q2.1 (G), R10.1
- new net: Q2.2 (D), Q3.2 (D)
- new net: Q3.1 (G), R13.1
- new net: Q1.1 (G), R3.1
- new net: D1.2 (A), D3.2 (A), Q1.2 (S), Q4.2 (S), R1.1, R12.2, R17.1
- new net: Q1.3 (D), R10.2, R4.2
- new net: Q4.1 (G), R15.2
- new net: Q4.3 (D), R13.2, R14.2
- new net: C4.2, R9.2, U1.17 (VC0)
- new net: C14.2, U1.3 (VSS)
- new net: R19.2, R20.1, U2.4 (ADJ)
- new net: C19.1, D6.2 (A), R19.1, U2.5 (VOUT)
- new net: D2.1 (K), R11.1, R18.1
- new net: C10.1, C11.2
- new net: C3.2, C8.1
- new net BAT: C14.1, R18.2, U1.10 (BAT), U1.9 (REGSRC)
- new net BAT+: C3.1, D2.2 (A), F1.1, Q2.3 (S), R11.2, R4.1
- new net BAT1P: J1.2 (Pin_2), J1.3 (Pin_3), R8.1
- new net BAT2P: J1.4 (Pin_4), J1.5 (Pin_5), R7.1
- new net BAT3P: F1.2, J1.6 (Pin_6), R6.1
- new net BATNOUT: C11.1, C2.2, D4.2 (A2), J2.2 (Pin_2), R5.1, U1.19 (SRN)
- new net BATPOUT: C10.2, C15.1, C18.2, C8.2, D4.1 (A1), J2.1 (Pin_1), M1.4 (VS), Q3.3 (S), R14.1, U2.1 (VIN), U2.3 (EN)
- new net CHG: D3.1 (K), R15.1, R17.2, U1.2 (CHG)
- new net DSG: D1.1 (K), R1.2, R3.2, U1.1 (DSG)
- new net REGOUT: C13.1, D6.1 (A), U1.8 (REGOUT)
- new net SCL: R22.2, U1.5 (SCL), U3.19 (PC1)
- new net SDA: R23.2, U1.4 (SDA), U3.18 (PC0)
- new net TS1: D5.1 (K), U1.6 (TS1)
- new net VDD: C16.1, C17.1, D6.3 (K), J3.1 (Pin_1), M1.2 (VSO), R22.1, R23.1, R24.2, R26.2, RV1.1, U3.8 (VDD)
- no-connect marks 8 -> 5
Other:
- note removed: "Debug Connection \nFor Programming and Debug"
- note removed: "IFX9201SG\nIntegrated MOSFET H-Bridge \nFor Driving Inductive loads upto 6A\nWith Direction and PWM Speed Control\nDiagnostics over SPI"
- note removed: "Input Terminal: DC12V IN\nVoltage Regulator for 3.3V Supply"
- note removed: "Output Terminal: DC12V OUT\n"
- note removed: "Output Transverse Voltage Suppressor \nwith Aluminium Electrolytic Capacitor"
- note removed: "Rotary Horizontally Mounted Potentiometer"
- note removed: "STM8L051F3 \n8-bit Microcontroller with 8kb Flash\nConnections with IFX9201SG:\n1. Serial Peripheral Interface Bus\nFor Diagnostics\n2. PWM and DIR\nFor speed and direction control."

Commit message: Updated date and credentials
Parts:
- J1: footprint (none) -> TerminalBlocks_Phoenix:TerminalBlock_Phoenix_MKDS1.5-6pol
- J2, J4: footprint (none) -> TerminalBlocks_Phoenix:TerminalBlock_Phoenix_MKDS1.5-2pol
Changed lines of the file:
@@
 Sheet 1 1
 Title "ARTIFICIAL LIMB DRIVER CARD"
-Date "2018-03-13"
+Date "2018-04-08"
 Rev "0.1"
 Comp ""
-Comment1 "Checked : SParnerkar"
-Comment2 "Engineer : SParnerkar"
+Comment1 "Checked : mighty840"
+Comment2 "Engineer : mighty840"
 Comment3 ""
 Comment4 ""
@@
 F 0 "J1" H 1050 1750 50  0000 C CNN
 F 1 "Screw_Terminal_01x06" H 1050 1050 50  0000 C CNN
-F 2 "" H 1050 1450 50  0001 C CNN
+F 2 "TerminalBlocks_Phoenix:TerminalBlock_Phoenix_MKDS1.5-6pol" H 1050 1450 50  0001 C CNN
 F 3 "" H 1050 1450 50  0001 C CNN
 	1    1050 1450
@@
 F 0 "J4" H 10800 4650 50  0000 C CNN
 F 1 "Screw_Terminal_01x02" H 10800 4350 50  0000 C CNN
-F 2 "" H 10800 4550 50  0001 C CNN
+F 2 "TerminalBlocks_Phoenix:TerminalBlock_Phoenix_MKDS1.5-2pol" H 10800 4550 50  0001 C CNN
 F 3 "" H 10800 4550 50  0001 C CNN
 	1    10800 4550
@@
 F 0 "J2" H 6000 4750 50  0000 C CNN
 F 1 "Screw_Terminal_01x02" H 6000 4450 50  0000 C CNN
-F 2 "" H 6000 4650 50  0001 C CNN
+F 2 "TerminalBlocks_Phoenix:TerminalBlock_Phoenix_MKDS1.5-2pol" H 6000 4650 50  0001 C CNN
 F 3 "" H 6000 4650 50  0001 C CNN
 	1    6000 4650
